File: hardware/TempSens.kicad_sch (KiCad schematic)
At the start: 20 parts, among them IC1 UCC12040DVE, J1 Conn_01x04_Pin, U1 LM1117-Q1, U2 LM1117-Q1, U3 XISO6463DWR, U4 XISO6463DWR

Commit message: Added some comments
Other:
- note added: "PROVERITI VREDNOSTI KONDENZATORA"
Changed lines of the file:
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@@
-		)
-	)
-	(text "TREBA ODREDITI KOLIKI OSIGURAC JE POTREBAN\n"
-		(exclude_from_sim no)
-		(at 104.902 224.536 0)
-		(effects
-			(font
-				(size 1.27 1.27)
-			)
 		)
 	)
@@
 				(thickness 0.508)
 				(bold yes)
+			)
+		)
+	)
+	(text "PROVERITI VREDNOSTI KONDENZATORA\n"
+		(exclude_from_sim no)
+		(at 74.93 19.558 0)
+		(effects
+			(font
+				(size 1.27 1.27)
 			)
 		)
@@
 				(thickness 0.508)
 				(bold yes)
-			)
-		)
-	)
-	(text "TREBA ODREDITI KOLIKI OSIGURAC JE POTREBAN\n"
-		(exclude_from_sim no)
-		(at 104.902 219.456 0)
-		(effects
-			(font
-				(size 1.27 1.27)
 			)
 		)
@@
 		)
 	)
-	(text "TREBA ODREDITI KOLIKI OSIGURAC JE POTREBAN\n"
-		(exclude_from_sim no)
-		(at 104.902 221.996 0)
-		(effects
-			(font
-				(size 1.27 1.27)
-			)
-		)
-	)
 	(text "Power Supply & SPI Interface"
 		(exclude_from_sim no)
@@
 		)
 	)
+	(text "TREBA ODREDITI KOLIKI OSIGURAC JE POTREBAN\n"
+		(exclude_from_sim no)
+		(at 179.578 52.07 0)
+		(effects
+			(font
+				(size 1.27 1.27)
+			)
+		)
+	)
